File: mirte-master-v2/mirte-master-v2.kicad_pcb (KiCad board)
At the start: 4 copper layers, 90.1 x 80.1 mm, 38 parts, among them J10 IMU MPU-9250, J11 Conn_01x03_Pin, J12 Conn_01x03_Pin, J13 sc, J14 sc, J16 sc, J17 sc, J18 sc, J19 sc, J20 sc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

Commit message: integrated the ina226 in the pcb layout
Parts:
- removed J20, J22: sc, easyeda:CONN-TH_XY126V-5.0-2P
- removed J7: INA226, Connector_JST:JST_XH_B4B-XH-A_1x04_P2.50mm_Vertical
- added C8: 100nF, Capacitor_SMD:C_0805_2012Metric, F.Cu at (116.3, 82.7)
- added C9: 100nF, Capacitor_SMD:C_0805_2012Metric, F.Cu at (112.3, 86.2)
- added JP1: SolderJumper_3_Bridged12, Jumper:SolderJumper-3_P1.3mm_Bridged12_RoundedPad1.0x1.5mm, F.Cu at (116.3, 91.2)
- added JP3: SolderJumper_3_Bridged12, Jumper:SolderJumper-3_P1.3mm_Bridged12_RoundedPad1.0x1.5mm, F.Cu at (119.4, 91.2)
- added R2: 2mR, Resistor_SMD:R_2512_6332Metric, F.Cu at (104.4, 86.2)
- added R3: 4R7, Resistor_SMD:R_0805_2012Metric, F.Cu at (109.3, 87.7)
- added R4: 4R7, Resistor_SMD:R_0805_2012Metric, F.Cu at (109.3, 84.7)
- added U1: INA226, Package_SO:VSSOP-10_3x3mm_P0.5mm, F.Cu at (117.3, 85.7)
- moved C3 6.95 mm to (110.0, 74.8), turned to -45 degrees
Connections:
- net -BATT renamed GND
Routing:
- net /power_input/SWITCHED_PWR: track 0.00 -> 15.9 mm
- net Net-(JP1-C): track 0.00 -> 9.30 mm
- net +5V: track 20.6 -> 28.3 mm, vias 4 -> 6
- net Net-(JP3-C): track 0.00 -> 7.45 mm
- net Net-(U1-Vin-): track 0.00 -> 5.51 mm
- net Net-(U1-Vin+): track 0.00 -> 5.30 mm
- net /SDA: track 82.7 -> 77.4 mm
- net +12V: track 2.43 -> 7.66 mm
- net /SCL: track 83.0 -> 78.2 mm
- net GND: track 3.05 -> 7.24 mm, vias 24 -> 25
- net /LED_STRIP: track 50.8 -> 53.6 mm
- added copper zone on In2.Cu, net +5V
Other:
- board text added: "MIRTE-Master: Compute V${VERSION}"
- board text removed: "12V GND GND SW_PWR"
- board text removed: "INA226 CURRENT SENSOR"
- board text removed: "MIRTE-Master: Compute V0.2+"
- board text removed: "SCL SDA GND 5V"
